File: Uno/kicad_project/Uno.kicad_sch (KiCad schematic)
At the start: 131 parts, among them J1 MC-318, J2 AFC12-S02DCC-00, J4 Fan, Q1 DDTA143ECA-7-F, Q2 DMP3099L-7, Q3 DDTA143ECA-7-F, Q4 SIS427EDN-T1-GE3, Q5 DMP3099L-7, Q6 ZXMN6A07FTA_C5122066, Q7 ZXMN6A07FTA_C5122066, T1 NEO-M8M-0, U1 FSUSB42UMX, U10 AZ1117CR2-3_3TRG1, U2 TJA1042TK_3_1J, U25 MT9700, U3 SY8368AQQC, U30 TJA1042TK_3_1J, U4 SY8368AQQC, U45 TJA1042TK_3_1J, U46 TJA1042TK_3_1J, U5 TPS92511DDAR, U6 TS-1087S-01526, U7 STM32F413RGTx, X1 U_FL-R-SMT-1(10), Y1 X322516MRB4SI, Y2 SC-32S32_768kHz20PPM12_5pF

Commit message: update of images and docs
Parts:
- D4: value BZT52C10 -> NRVB130T1G
Changed lines of the file:
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@@
       (effects (font (size 1.27 1.27)) (justify left))
     )
-    (property "Value" "BZT52C10" (at 359.283 342.773 90)
+    (property "Value" "NRVB130T1G" (at 359.283 342.773 90)
       (effects (font (size 1.27 1.27)) (justify left))
     )
