File: BlackPanda/kicad_project/BlackPanda.kicad_pcb (KiCad board)
At the start: 4 copper layers, 47.5 x 41.7 mm, 86 parts, among them P1 TYPE-C-31-M-04, Q1 DDTA143ECA-7-F P08, Q2 DDTA143ECA-7-F P08, Q3 PDTC114EU, Q4 HY12P03C2, SW1 SW_Push, U1 AP22615AWU-7, U10 TJA1042TK-3, U11 TJA1042TK-3, U12 XL1509-3.3, U2 SiP32431DR3, U3 10_0_QHHTZB6_3, U4 NEO-M8M, U5 FM-B1921RGBA-SH, U6 TPS5450DDAR, U7 STM32F413RGTx, U8 TJA1042TK-3, U9 TJA1042TK-3, Y1 X322516MLB4SI

Commit message: CAN labels mirrored and rotated according to USB-C cables connections
Connections:
- D6 pad 1: CAN0_L -> CAN1_L
- D6 pad 2: CAN0_H -> CAN1_H
- D7 pad 1: CAN1_L -> CAN0_L
- D7 pad 2: CAN1_H -> CAN0_H
- D8 pad 1: CAN2_L -> CAN3_L
- D8 pad 2: CAN2_H -> CAN3_H
- D9 pad 1: CAN3_L -> CAN2_L
- D9 pad 2: CAN3_H -> CAN2_H
- P1 pad A10: CAN1_L -> CAN0_L
- P1 pad A11: CAN1_H -> CAN0_H
- P1 pad A2: CAN0_H -> CAN1_H
- P1 pad A3: CAN0_L -> CAN1_L
- P1 pad B10: CAN3_L -> CAN2_L
- P1 pad B11: CAN3_H -> CAN2_H
- P1 pad B2: CAN2_H -> CAN3_H
- P1 pad B3: CAN2_L -> CAN3_L
- U10 pad 1: CAN2_TX -> CAN3_TX
- U10 pad 4: CAN2_RX -> CAN3_RX
- U10 pad 6: CAN2_L -> CAN3_L
- U10 pad 7: CAN2_H -> CAN3_H
- U10 pad 8: CAN2_EN -> CAN3_EN
- U11 pad 1: CAN3_TX -> CAN2_TX
- U11 pad 4: CAN3_RX -> CAN2_RX
- U11 pad 6: CAN3_L -> CAN2_L
- U11 pad 7: CAN3_H -> CAN2_H
- U11 pad 8: CAN3_EN -> CAN2_EN
- U7 pad 14: CAN1_EN -> CAN0_EN
- U7 pad 2: CAN2_EN -> CAN3_EN
- U7 pad 29: CAN0_EN -> CAN1_EN
- U7 pad 33: CAN0_RX -> CAN1_RX
- U7 pad 34: CAN0_TX -> CAN1_TX
- U7 pad 41: CAN1_RX -> CAN0_RX
- U7 pad 50: CAN1_TX -> CAN0_TX
- U7 pad 57: CAN2_RX -> CAN3_RX
- U7 pad 58: CAN2_TX -> CAN3_TX
- U7 pad 61: CAN3_RX -> CAN2_RX
- U7 pad 62: CAN3_TX -> CAN2_TX
- U7 pad 9: CAN3_EN -> CAN2_EN
- U8 pad 1: CAN0_TX -> CAN1_TX
- U8 pad 4: CAN0_RX -> CAN1_RX
- U8 pad 6: CAN0_L -> CAN1_L
- U8 pad 7: CAN0_H -> CAN1_H
- U8 pad 8: CAN0_EN -> CAN1_EN
- U9 pad 1: CAN1_TX -> CAN0_TX
- U9 pad 4: CAN1_RX -> CAN0_RX
- U9 pad 6: CAN1_L -> CAN0_L
- U9 pad 7: CAN1_H -> CAN0_H
- U9 pad 8: CAN1_EN -> CAN0_EN
Routing:
- net CAN3_TX: track 49.2 -> 31.3 mm
- net CAN2_TX: track 31.3 -> 49.2 mm
- net CAN3_RX: track 52.4 -> 34.6 mm
- net CAN2_RX: track 34.6 -> 52.4 mm
- net CAN3_L: track 10.0 -> 20.5 mm
- net CAN2_L: track 20.5 -> 10.0 mm
- net CAN3_H: track 8.96 -> 18.8 mm
- net CAN2_H: track 18.8 -> 8.96 mm
- net CAN1_TX: track 18.1 -> 26.8 mm, vias 0 -> 2
- net CAN0_TX: track 26.8 -> 18.1 mm, vias 2 -> 0
- net CAN1_L: track 5.85 -> 13.6 mm
- net CAN0_L: track 13.6 -> 5.85 mm
- net CAN1_H: track 7.34 -> 12.1 mm
- net CAN0_H: track 12.1 -> 7.34 mm
- net CAN1_EN: track 29.0 -> 31.7 mm
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